File: schematics/adc.kicad_sch (KiCad schematic)
At the start: 19 parts

Commit message: cleanup, fixes, started on power supplies
Parts:
- removed C?: ~, symbol Device:C_Small
- added C43: 0u1, symbol Device:C_Small
- added R54: 9k, symbol Device:R_Small
- added R55: 1k, symbol Device:R_Small
- C45: renamed from C?; value ~ -> 0u22
- C46, C47: renamed from C?; value ~ -> 1u
- D11: renamed from D?; value ~ -> 6.2V
- D12: renamed from D?; footprint (none) -> Diode_THT:D_DO-35_SOD27_P7.62mm_Horizontal
- IC30: renamed from U?; value ~ -> ICL7135
- IC34: renamed from U?; value ~ -> MUX24
- R33: renamed from R?; value ~ -> 1k
- R34: renamed from R?; value ~ -> 19R
- R36: renamed from R?; value ~ -> 10k
- R39, R48: renamed from R?; value ~ -> 1k96
- R40, R44: renamed from R?; value ~ -> 97k6
- gave numbers to parts that had none: 4
Connections:
- net AVEE: now also IC34.3 (V-); no longer IC34. (V-)
- net GND: now also IC34.15 (GND), C43.2, R55.2
- net REF: now also R54.1; no longer IC30.2 (REF)
- net VCC: now also C43.1
- net at IC30.10 (IN+): now also IC34.9 (OB); no longer IC34. (V-)
- net at IC30.9 (IN-): now also IC34.8 (OA); no longer IC34. (V-)
- new net: IC30.2 (REF), R54.2, R55.1

Commit message: More power supply work
Connections:
- net S0 renamed D0
- net S1 renamed D1

Commit message: Updated to KiCad v10.0. Minor improvements.
Parts:
- C64, D12, R31, RV3, RV4: value ~ -> (none)
