File: schematics/display.kicad_sch (KiCad schematic)
At the start: 0 parts

Commit message: More power supply work
Parts:
- added IC1, IC5: ULN2803A, symbol Transistor_Array:ULN2803A
- added IC2, IC7: 74LS259, symbol 74xx:74LS259
- added IC3, IC6: A2982, Package_SO:SOIC-20W_7.5x12.8mm_P1.27mm, symbol Transistor_Array:A2982
- added IC4: 74LS374, symbol 74xx:74LS374
- added J?: ~, symbol Connector:Conn_01x18_Male
- added LED1, LED10, LED18, LED2, LED3, LED4: HLMP-5635, symbol Custom:HLMP-5635
- added LED11, LED12, LED19, LED20: HLMP-5300, symbol Custom:HLMP-5300
- added LED13, LED5: 5082-H, symbol Custom:5082-H
- added LED6, LED7, LED8, LED9, LED? (x4): 5082-F, symbol Custom:5082-F
- added RP1, RP2, RP3: 470Ω, symbol Device:R_Pack08
- added RP4: 1kΩ, symbol Device:R_Pack08
Connections:
- new net: LED12.1, RP3.4 (R4.1)
- new net: LED12.2, LED12.3
- new net: LED13.1, LED5.1, RP4.11 (R6.2)
- new net: LED13.10, LED5.10, RP4.14 (R3.2)
- new net: LED13.3, LED5.3, RP4.10 (R7.2)
- new net: LED13.4, LED5.4, RP4.9 (R8.2)
- new net: LED13.8, LED5.8, RP4.12 (R5.2)
- new net: LED13.9, LED5.9, RP4.13 (R4.2)
- new net: IC1.11 (O8), RP1.1 (R1.1)
- new net: IC1.12 (O7), RP1.2 (R2.1)
- new net: IC1.13 (O6), RP1.4 (R4.1)
- new net: IC1.14 (O5), RP1.7 (R7.1)
- new net: IC1.15 (O4), RP1.8 (R8.1)
- new net: IC1.16 (O3), RP1.3 (R3.1)
- new net: IC1.17 (O2), RP1.5 (R5.1)
- new net: IC1.18 (O1), RP1.6 (R6.1)
- new net: IC2.4 (Q0), IC3.1 (IN1)
- new net: IC2.5 (Q1), IC3.2 (IN2)
- new net: IC2.6 (Q2), IC3.3 (IN3)
- new net: IC2.7 (Q3), IC3.4 (IN4)
- new net: IC2.9 (Q4), IC3.5 (IN5)
- new net: IC2.10 (Q5), IC3.6 (IN6)
- new net: IC2.11 (Q6), IC3.7 (IN7)
- new net: IC2.12 (Q7), IC3.8 (IN8)
- new net: LED2.1, LED2.3
- new net: LED2.10, LED2.12
- new net: LED2.11, LED2.13
- new net: LED2.4, LED2.6
- new net: LED2.5, LED2.7
- new net: LED1.9, LED10.9, LED18.9, LED2.8, RP2.6 (R6.1), RP2.7 (R7.1)
- new net: LED18.8, LED2.9, LED3.8, RP2.4 (R4.1), RP2.5 (R5.1)
- new net: LED4.9, RP2.1 (R1.1)
- new net: IC5.15 (O4), IC5.17 (O2), RP2.10 (R7.2), RP2.12 (R5.2), RP4.3 (R3.1), RP4.4 (R4.1), RP4.5 (R5.1)
- new net: IC5.16 (O3), IC5.18 (O1), RP2.11 (R6.2), RP2.9 (R8.2), RP4.6 (R6.1), RP4.7 (R7.1), RP4.8 (R8.1)
- new net: IC5.14 (O5), RP2.13 (R4.2), RP3.13 (R4.2)
- new net: IC5.13 (O6), RP2.14 (R3.2), RP3.14 (R3.2)
- new net: IC5.12 (O7), RP2.15 (R2.2), RP3.15 (R2.2)
- new net: IC5.11 (O8), RP2.16 (R1.2), RP3.16 (R1.2)
- new net: LED4.8, RP2.2 (R2.1)
- new net: LED3.9, RP2.3 (R3.1)
- new net: LED1.8, LED10.8, RP2.8 (R8.1)
- new net: IC6.1 (IN1), IC7.4 (Q0)
- new net: IC6.2 (IN2), IC7.5 (Q1)
- new net: IC6.3 (IN3), IC7.6 (Q2)
- new net: IC6.4 (IN4), IC7.7 (Q3)
- new net: IC4.2 (O0), IC5.1 (I1)
- new net: IC4.5 (O1), IC5.2 (I2)
- new net: IC4.6 (O2), IC5.3 (I3)
- new net: IC4.9 (O3), IC5.4 (I4)
- new net: IC4.12 (O4), IC5.5 (I5)
- new net: IC4.15 (O5), IC5.6 (I6)
- new net: IC4.16 (O6), IC5.7 (I7)
- new net: IC4.19 (O7), IC5.8 (I8)
- new net: LED3.1, LED3.3
- new net: LED3.10, LED3.12
- new net: LED3.11, LED3.13
- new net: LED3.14, LED3.16
- new net: LED3.4, LED3.6
- new net: LED3.5, LED3.7
- new net: LED19.1, RP3.1 (R1.1)
- new net: LED20.1, RP3.2 (R2.1)
- new net: LED11.1, RP3.3 (R3.1)
- new net: LED18.1, LED18.3
- new net: LED18.10, LED18.12
- new net: LED18.11, LED18.13
- new net: LED18.14, LED18.16
- new net: LED18.4, LED18.6
- new net: LED18.5, LED18.7
- new net: LED1.1, LED1.3
- new net: LED1.10, LED1.12
- new net: LED1.11, LED1.13
- new net: LED1.4, LED1.6
- new net: LED1.5, LED1.7
- new net: LED11.2, LED11.3
- new net: LED19.2, LED19.3
- new net: LED4.1, LED4.3
- new net: LED4.10, LED4.12
- new net: LED4.11, LED4.13
- new net: LED4.14, LED4.16
- new net: LED4.4, LED4.6
- new net: LED4.5, LED4.7
- new net: LED10.1, LED10.3
- new net: LED10.10, LED10.12
- new net: LED10.11, LED10.13
- new net: LED10.14, LED10.16
- new net: LED10.4, LED10.6
- new net: LED10.5, LED10.7
- new net: LED20.2, LED20.3
- new net 22V5: IC1.10 (COM), IC3.9 (+VS), IC5.10 (COM), IC6.9 (+VS), J?.1 (Pin_1)
- new net 5V: IC2.13 (D), IC2.16 (VCC), IC4.20 (VCC), IC7.13 (D), IC7.16 (VCC), J?.2 (Pin_2)
- new net D0: IC3.20 (OUT1), LED6.11, LED6.3
- new net D1: IC3.19 (OUT2), LED7.11, LED7.3
- new net D10: IC6.18 (OUT3), LED5.11, LED5.12, LED5.2, LED5.5, LED5.6, LED5.7
- new net D11: IC6.17 (OUT4), LED13.11, LED13.12, LED13.2, LED13.5, LED13.6, LED13.7
- new net D2: IC3.18 (OUT3), LED8.11, LED8.3
- new net D3: IC3.17 (OUT4), LED9.11, LED9.3
- new net D4: IC3.16 (OUT5), LED?.11, LED?.3
- new net D5: IC3.15 (OUT6), LED?.11, LED?.3
- new net D6: IC3.14 (OUT7), LED?.11, LED?.3
- new net D7: IC3.13 (OUT8), LED?.11, LED?.3
- new net D8: IC6.20 (OUT1), LED1.14, LED1.15, LED1.16, LED1.2, LED2.14, LED2.15, LED2.16, LED2.2, LED3.15, LED3.2, LED4.15, LED4.2
- new net D9: IC6.19 (OUT2), LED10.15, LED10.2, LED11.4, LED12.4, LED18.15, LED18.2, LED19.4, LED20.4
- new net DSP10: IC4.11 (Cp), J?.10 (Pin_10)
- new net DSP11: IC1.8 (I8), IC4.18 (D7), J?.11 (Pin_11)
- new net DSP12: IC1.7 (I7), IC4.17 (D6), J?.12 (Pin_12)
- new net DSP13: IC1.6 (I6), IC4.14 (D5), J?.13 (Pin_13)
- new net DSP14: IC1.5 (I5), IC4.13 (D4), J?.14 (Pin_14)
- new net DSP15: IC1.4 (I4), IC4.8 (D3), J?.15 (Pin_15)
- new net DSP16: IC1.3 (I3), IC4.7 (D2), J?.16 (Pin_16)
- new net DSP17: IC1.2 (I2), IC4.4 (D1), J?.17 (Pin_17)
- new net DSP18: IC1.1 (I1), IC4.3 (D0), J?.18 (Pin_18)
- new net DSP3: IC1.9 (GND), IC2.15 (Clr), IC2.8 (GND), IC3.12 (GND), IC4.1 (OE), IC4.10 (GND), IC5.9 (GND), IC6.12 (GND), IC7.15 (Clr), IC7.3 (A2), IC7.8 (GND), J?.3 (Pin_3)
- new net DSP4: IC2.1 (A0), J?.4 (Pin_4)
- new net DSP5: IC2.2 (A1), J?.5 (Pin_5)
- new net DSP6: IC2.3 (A2), J?.6 (Pin_6)
- new net DSP7: IC2.14 (E), IC7.14 (E), J?.7 (Pin_7)
- new net DSP8: IC7.1 (A0), J?.8 (Pin_8)
- new net DSP9: IC7.2 (A1), J?.9 (Pin_9)
- new net S0: LED6.1, LED7.1, LED8.1, LED9.1, LED?.1, LED?.1, LED?.1, LED?.1, RP1.16 (R1.2)
- new net S1: LED6.10, LED7.10, LED8.10, LED9.10, LED?.10, LED?.10, LED?.10, LED?.10, RP1.15 (R2.2)
- new net S2: LED6.2, LED7.2, LED8.2, LED9.2, LED?.2, LED?.2, LED?.2, LED?.2, RP1.14 (R3.2)
- new net S3: LED6.9, LED7.9, LED8.9, LED9.9, LED?.9, LED?.9, LED?.9, LED?.9, RP1.13 (R4.2)
- new net S4: LED6.8, LED7.8, LED8.8, LED9.8, LED?.8, LED?.8, LED?.8, LED?.8, RP1.12 (R5.2)
- new net S5: LED6.7, LED7.7, LED8.7, LED9.7, LED?.7, LED?.7, LED?.7, LED?.7, RP1.11 (R6.2)
- new net S6: LED6.6, LED7.6, LED8.6, LED9.6, LED?.6, LED?.6, LED?.6, LED?.6, RP1.10 (R7.2)
- new net S7: LED6.5, LED7.5, LED8.5, LED9.5, LED?.5, LED?.5, LED?.5, LED?.5, RP1.9 (R8.2)
- no-connect marks 0 -> 28

Commit message: Updated to KiCad v10.0. Minor improvements.
Parts:
- J?: value ~ -> (none)
