File: schematics/gpib_ctrl_acia.kicad_sch (KiCad schematic)
At the start: 0 parts

Commit message: Moved more components into hierachical sheets, misc cleanup
Parts:
- added R?: 560, symbol Device:R_Small
- added R?: 330, symbol Device:R_Small
- added U?: MC68A50, Package_DIP:DIP-40_W15.24mm, symbol Interface_UART:MC68A50
- added U?: HCPL-2601, Package_DIP:DIP-8_W7.62mm, symbol Isolator:HCPL-2601
- added U?: 74LS04, symbol Custom:74LS04
Connections:
- new net: U?.12 (6Y), U?.2 (Rx_Data)
- new net: U?.11 (5A), U?.6 (Tx_Data)
- new net: U?.10 (5Y), U?.2 (A)
- new net: R?.1, U?.3 (C)
- new net A0: U?.11 (RS)
- new net A5: U?.10 (CS1)
- new net A6: U?.8 (CS0)
- new net CS: U?.9 (CS2)
- new net D0: U?.22 (D0)
- new net D1: U?.21 (D1)
- new net D2: U?.20 (D2)
- new net D3: U?.19 (D3)
- new net D4: U?.18 (D4)
- new net D5: U?.17 (D5)
- new net D6: U?.16 (D6)
- new net D7: U?.15 (D7)
- new net E: U?.14 (E), U?.3 (Rx_CLK), U?.4 (Tx_CLK)
- new net GND: R?.2, R?.2, U?.1 (VSS), U?.23 (~{DCD}), U?.24 (~{CTS}), U?.5 (GND), U?.7 (VEE)
- new net R/~{W}: U?.13 (R/~{W})
- new net VCC: U?.12 (VCC), U?.14 (VCC), U?.8 (VCC)
- new net ~{IRQ}: U?.7 (~{IRQ})
- new net ~{RX}: R?.1, U?.13 (6A)
- new net ~{TX}: U?.6 (VO)
- no-connect marks 0 -> 10

Commit message: cleanup, fixes, started on power supplies
Parts:
- removed R?: 560, symbol Device:R_Small
- removed U?: HCPL-2601, Package_DIP:DIP-8_W7.62mm, symbol Isolator:HCPL-2601
- added C10, C11: .1u, symbol Device:C_Small
- gave numbers to parts that had none: 3
Connections:
- net GND: now also C10.2, C11.2
- net VCC: now also C10.1, C11.1
- net ~{TX}: now also IC10.10 (5Y)
- net RX: now reaches IC10.12 (6Y), IC11.2 (Rx_Data)
- no-connect marks 10 -> 9

Commit message: More power supply work
Parts:
- IC10: value 74LS04 -> 74LD04
Connections:
- net A5 renamed A7
