File: schematics/gpib_ctrl_reg_and_reset.kicad_sch (KiCad schematic)
At the start: 7 parts

Commit message: cleanup, fixes, started on power supplies
Parts:
- gave numbers to parts that had none: 6
Other:
- moved on the sheet: C76, C77
Changed lines of the file:
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@@
 (kicad_sch (version 20211123) (generator eeschema)
   (paper "A4")
-  (junction (at 124.46 142.24) (diameter 0) (color 0 0 0 0)
-  )
-  (junction (at 124.46 111.76) (diameter 0) (color 0 0 0 0)
-  )
   (junction (at 101.6 86.36) (diameter 0) (color 0 0 0 0)
   )
@@
   (junction (at 154.94 142.24) (diameter 0) (color 0 0 0 0)
   )
+  (junction (at 121.92 142.24) (diameter 0) (color 0 0 0 0)
+  )
   (junction (at 124.46 116.84) (diameter 0) (color 0 0 0 0)
   )
   (junction (at 124.46 124.46) (diameter 0) (color 0 0 0 0)
   )
+  (junction (at 121.92 111.76) (diameter 0) (color 0 0 0 0)
+  )
   (junction (at 101.6 55.88) (diameter 0) (color 0 0 0 0)
   )
@@
     (stroke (width 0) (type default) (color 0 0 0 0))
   )
-  (wire (pts (xy 124.46 134.62) (xy 127 134.62))
+  (wire (pts (xy 121.92 134.62) (xy 127 134.62))
     (stroke (width 0) (type default) (color 0 0 0 0))
   )
@@
     (stroke (width 0) (type default) (color 0 0 0 0))
   )
+  (wire (pts (xy 121.92 111.76) (xy 139.7 111.76))
+    (stroke (width 0) (type default) (color 0 0 0 0))
+  )
   (wire (pts (xy 119.38 55.88) (xy 167.64 55.88))
     (stroke (width 0) (type default) (color 0 0 0 0))
@@
     (stroke (width 0) (type default) (color 0 0 0 0))
   )
-  (wire (pts (xy 124.46 111.76) (xy 139.7 111.76))
-    (stroke (width 0) (type default) (color 0 0 0 0))
-  )
   (wire (pts (xy 111.76 63.5) (xy 111.76 111.76))
     (stroke (width 0) (type default) (color 0 0 0 0))
@@
     (stroke (width 0) (type default) (color 0 0 0 0))
   )
-  (wire (pts (xy 124.46 109.22) (xy 124.46 111.76))
+  (wire (pts (xy 121.92 109.22) (xy 121.92 111.76))
     (stroke (width 0) (type default) (color 0 0 0 0))
   )
@@
     (stroke (width 0) (type default) (color 0 0 0 0))
   )
-  (wire (pts (xy 124.46 139.7) (xy 124.46 142.24))
-    (stroke (width 0) (type default) (color 0 0 0 0))
-  )
-  (wire (pts (xy 124.46 104.14) (xy 127 104.14))
+  (wire (pts (xy 121.92 139.7) (xy 121.92 142.24))
+    (stroke (width 0) (type default) (color 0 0 0 0))
+  )
+  (wire (pts (xy 121.92 104.14) (xy 127 104.14))
     (stroke (width 0) (type default) (color 0 0 0 0))
   )
@@
     (stroke (width 0) (type default) (color 0 0 0 0))
   )
+  (wire (pts (xy 121.92 142.24) (xy 139.7 142.24))
+    (stroke (width 0) (type default) (color 0 0 0 0))
+  )
   (wire (pts (xy 154.94 142.24) (xy 139.7 142.24))
     (stroke (width 0) (type default) (color 0 0 0 0))
@@
     (stroke (width 0) (type default) (color 0 0 0 0))
   )
-  (wire (pts (xy 111.76 142.24) (xy 124.46 142.24))
+  (wire (pts (xy 111.76 142.24) (xy 121.92 142.24))
     (stroke (width 0) (type default) (color 0 0 0 0))
   )
@@
     (stroke (width 0) (type default) (color 0 0 0 0))
   )
-  (wire (pts (xy 124.46 142.24) (xy 139.7 142.24))
-    (stroke (width 0) (type default) (color 0 0 0 0))
-  )
-  (wire (pts (xy 111.76 111.76) (xy 124.46 111.76))
+  (wire (pts (xy 111.76 111.76) (xy 121.92 111.76))
     (stroke (width 0) (type default) (color 0 0 0 0))
   )
@@
   (symbol (lib_id "Power_Supervisor:TL7705A") (at 139.7 99.06 0) (unit 1)
     (in_bom yes) (on_board yes) (fields_autoplaced)
-    (property "Reference" "U?" (id 0) (at 141.7194 86.36 0)
+    (property "Reference" "U41" (id 0) (at 141.7194 86.36 0)
       (effects (font (size 1.27 1.27)) (justify left))
     )
@@
   (symbol (lib_id "Regulator_Linear:L7805") (at 111.76 55.88 0) (unit 1)
     (in_bom yes) (on_board yes) (fields_autoplaced)
-    (property "Reference" "U?" (id 0) (at 111.76 48.895 0))
-    (property "Value" "L7805" (id 1) (at 111.76 51.435 0))
+    (property "Reference" "REG1" (id 0) (at 111.76 48.26 0))
+    (property "Value" "L7805" (id 1) (at 111.76 50.8 0))
     (property "Footprint" "" (id 2) (at 112.395 59.69 0)
       (effects (font (size 1.27 1.27) italic) (justify left) hide)
@@
   (symbol (lib_id "Device:C_Small") (at 154.94 137.16 0) (unit 1)
     (in_bom yes) (on_board yes) (fields_autoplaced)
-    (property "Reference" "C?" (id 0) (at 157.48 135.8962 0)
+    (property "Reference" "C74" (id 0) (at 157.48 135.8962 0)
       (effects (font (size 1.27 1.27)) (justify left))
     )
@@
     (pin "2")
   )
-  (symbol (lib_id "Device:C_Small") (at 124.46 106.68 0) (unit 1)
-    (in_bom yes) (on_board yes) (fields_autoplaced)
-    (property "Reference" "C?" (id 0) (at 127 105.4162 0)
-      (effects (font (size 1.27 1.27)) (justify left))
-    )
-    (property "Value" "4.7u" (id 1) (at 127 107.9562 0)
-      (effects (font (size 1.27 1.27)) (justify left))
-    )
-    (property "Footprint" "" (id 2) (at 124.46 106.68 0)
-      (effects (font (size 1.27 1.27)) hide)
-    )
-    (property "Datasheet" "~" (id 3) (at 124.46 106.68 0)
-      (effects (font (size 1.27 1.27)) hide)
-    )
-    (pin "1")
-    (pin "2")
-  )
-  (symbol (lib_id "Device:C_Small") (at 124.46 137.16 0) (unit 1)
-    (in_bom yes) (on_board yes) (fields_autoplaced)
-    (property "Reference" "C?" (id 0) (at 127 135.8962 0)
-      (effects (font (size 1.27 1.27)) (justify left))
-    )
-    (property "Value" "470n" (id 1) (at 127 138.4362 0)
-      (effects (font (size 1.27 1.27)) (justify left))
-    )
-    (property "Footprint" "" (id 2) (at 124.46 137.16 0)
-      (effects (font (size 1.27 1.27)) hide)
-    )
-    (property "Datasheet" "~" (id 3) (at 124.46 137.16 0)
+  (symbol (lib_id "Device:C_Small") (at 121.92 106.68 0) (unit 1)
+    (in_bom yes) (on_board yes) (fields_autoplaced)
+    (property "Reference" "C76" (id 0) (at 124.46 105.4162 0)
+      (effects (font (size 1.27 1.27)) (justify left))
+    )
+    (property "Value" "4.7u" (id 1) (at 124.46 107.9562 0)
+      (effects (font (size 1.27 1.27)) (justify left))
+    )
+    (property "Footprint" "" (id 2) (at 121.92 106.68 0)
+      (effects (font (size 1.27 1.27)) hide)
+    )
+    (property "Datasheet" "~" (id 3) (at 121.92 106.68 0)
+      (effects (font (size 1.27 1.27)) hide)
+    )
+    (pin "1")
+    (pin "2")
+  )
+  (symbol (lib_id "Device:C_Small") (at 121.92 137.16 0) (unit 1)
+    (in_bom yes) (on_board yes) (fields_autoplaced)
+    (property "Reference" "C77" (id 0) (at 124.46 135.8962 0)
+      (effects (font (size 1.27 1.27)) (justify left))
+    )
+    (property "Value" "470n" (id 1) (at 124.46 138.4362 0)
+      (effects (font (size 1.27 1.27)) (justify left))
+    )
+    (property "Footprint" "" (id 2) (at 121.92 137.16 0)
+      (effects (font (size 1.27 1.27)) hide)
+    )
+    (property "Datasheet" "~" (id 3) (at 121.92 137.16 0)
       (effects (font (size 1.27 1.27)) hide)
     )
@@
   (symbol (lib_id "Device:C_Small") (at 154.94 106.68 0) (unit 1)
     (in_bom yes) (on_board yes) (fields_autoplaced)
-    (property "Reference" "C?" (id 0) (at 157.48 105.4162 0)
-      (effects (font (size 1.27 1.27)) (justify left))
-    )
+    (property "Reference" "C75" (id 0) (at 157.48 105.4162 0)
+      (effects (font (size 1.27 1.27)) (justify left))
+    )

Commit message: Updated to KiCad v10.0. Minor improvements.
Connections:
- net GPIB_CTRL_UNREG renamed GPIB_CTRL_UNREG+
