File: schematics/gpib_interface.kicad_sch (KiCad schematic)
At the start: 0 parts

Commit message: Moved more components into hierachical sheets, misc cleanup
Parts:
- added R?: 10k, symbol Device:R_Small
- added RN?: 10k, Resistor_THT:R_Array_SIP7, symbol Device:R_Network06
- added SW?: SW_DIP_x06, symbol Switch:SW_DIP_x06
- added U?: MC68488, symbol Custom:MC68488
- added U?: 74LS366, symbol 74xx:74LS366
- added U? (x2): MC3447, symbol Custom:MC3447
Connections:
- new net: RN?.4 (R3), SW?.10, U?.6 (I3)
- new net: RN?.3 (R2), SW?.11, U?.4 (I2)
- new net: RN?.2 (R1), SW?.12, U?.2 (I1)
- new net: RN?.6 (R5), SW?.7, U?.12 (I5)
- new net: RN?.5 (R4), SW?.8, U?.10 (I4)
- new net: RN?.7 (R6), SW?.9, U?.14 (I6)
- new net: U?.15 (E2), U?.4 (~{ASE})
- new net A0: U?.37 (RS0)
- new net A1: U?.38 (RS1)
- new net A2: U?.39 (RS2)
- new net B0: U?.22 (B1)
- new net B1: U?.22 (B1)
- new net B10: U?.18 (B5)
- new net B11: U?.18 (B5)
- new net B12: U?.15 (B7)
- new net B13: U?.23 (B0)
- new net B14: U?.16 (B6)
- new net B15: U?.15 (B7)
- new net B2: U?.21 (B2)
- new net B3: U?.21 (B2)
- new net B4: U?.20 (B3)
- new net B5: U?.20 (B3)
- new net B6: U?.19 (B4)
- new net B7: U?.19 (B4)
- new net B8: U?.16 (B6)
- new net B9: U?.23 (B0)
- new net CS: U?.3 (~{CS})
- new net D0: U?.3 (O1), U?.7 (D0)
- new net D1: U?.5 (O2), U?.8 (D1)
- new net D2: U?.7 (O3), U?.9 (D2)
- new net D3: U?.10 (D3), U?.11 (O5)
- new net D4: U?.11 (D4), U?.13 (O6)
- new net D5: U?.12 (D5), U?.9 (O4)
- new net D6: U?.13 (D6)
- new net D7: U?.14 (D7)
- new net E: U?.6 (E)
- new net GND: SW?.1, SW?.2, SW?.3, SW?.4, SW?.5, SW?.6, U?. (VSS), U?. (VSS), U?.1 (E1), U?.1 (EN_0), U?.1 (VEE), U?.11 (EN_6), U?.14 (EN_7), U?.14 (EN_7), U?.8 (GND)
- new net GPIB_GND: U?. (VSS), U?. (VSS)
- new net IATN: U?.26 (~{ATN}), U?.9 (D6)
- new net IB0: U?.3 (D1), U?.36 (~{B0})
- new net IB1: U?.3 (D1), U?.35 (~{B1})
- new net IB10: U?.18 (RFD), U?.7 (D5)
- new net IB11: U?.17 (DAC), U?.7 (D5)
- new net IB12: U?.10 (D7), U?.21 (~{IFC})
- new net IB13: R?.2, U?.2 (D0), U?.23 (~{SRQ})
- new net IB15: U?.10 (D7), U?.22 (~{REN})
- new net IB2: U?.34 (~{B2}), U?.4 (D2)
- new net IB3: U?.33 (~{B3}), U?.4 (D2)
- new net IB4: U?.32 (~{B4}), U?.5 (D3)
- new net IB5: U?.31 (~{}B5), U?.5 (D3)
- new net IB6: U?.30 (~{B6}), U?.6 (D4)
- new net IB7: U?.29 (~{B7}), U?.6 (D4)
- new net IB8: U?.25 (~{EOI}), U?.9 (D6)
- new net IB9: U?.16 (~{DAV}), U?.2 (D0)
- new net R/~{W}: U?.5 (R/W)
- new net T/R1: U?.28 (T/R1)
- new net T/R2: U?.1 (EN_0), U?.11 (EN_6), U?.17 (EN_1-4), U?.17 (EN_1-4), U?.27 (T/R2), U?.8 (EN_5), U?.8 (EN_5)
- new net VCC: R?.1, RN?.1 (common), U?.16 (VCC), U?.2 (DMA_GRN), U?.20 (VCC), U?.24 (VCC), U?.24 (VCC)
- new net ~{RESET}: U?.19 (~{RESET})
- no-connect marks 0 -> 1

Commit message: cleanup, fixes, started on power supplies
Parts:
- added C1, C3, C4, C5: .1u, symbol Device:C_Small
- gave numbers to parts that had none: 7
Connections:
- net GND: now also C1.2, C3.2, C4.2, C5.2
- net VCC: now also C1.1, C3.1, C4.1, C5.1

Commit message: More power supply work
Parts:
- IC1: value 74LS366 -> 74LD366
