File: schematics/latched_dac.kicad_sch (KiCad schematic)
At the start: 2 parts

Commit message: cleanup, fixes, started on power supplies
Parts:
- gave numbers to parts that had none: 2
Changed lines of the file:
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@@
   (symbol (lib_id "74xx:74LS377") (at 109.22 93.98 0) (unit 1)
     (in_bom yes) (on_board yes)
-    (property "Reference" "U?" (id 0) (at 101.6 76.2 0)
+    (property "Reference" "IC27" (id 0) (at 101.6 76.2 0)
       (effects (font (size 1.27 1.27)) (justify left))
     )
@@
   (symbol (lib_id "Custom:DAC0801") (at 142.24 76.2 0) (unit 1)
     (in_bom yes) (on_board yes)
-    (property "Reference" "U?" (id 0) (at 140.97 77.47 0)
+    (property "Reference" "IC26" (id 0) (at 140.97 77.47 0)
       (effects (font (size 1.27 1.27)) (justify left))
     )

Commit message: More power supply work
Parts:
- added C?: C_Small, symbol Device:C_Small
- added R29: 5k11, symbol Device:R_Small
Connections:
- net VLC is gone; now on net GND: IC26.1 (VLC)
- net AVEE: now also C?.2
- net REF+: now also R29.2; no longer IC26.14 (R+)
- net COMP: no longer names the net of IC26.16 (CMP)
- net COMP: now also C?.1
- net VEE renamed GND
- new net: IC26.14 (R+), R29.1

Commit message: Updated to KiCad v10.0. Minor improvements.
Parts:
- IC26, IC27: value ~ -> (none)
