File: schematics/secondary_processor.kicad_sch (KiCad schematic)
At the start: 0 parts

Commit message: Moved more components into hierachical sheets, misc cleanup
Parts:
- added C? (x2): C_Small, symbol Device:C_Small
- added D? (x2): D_Small, symbol Device:D_Small
- added LK2: Conn_01x03_Male, symbol Connector:Conn_01x03_Male
- added R12: 1k, symbol Device:R_Small
- added R5, R6: 3k3, symbol Device:R_Small
- added R7: 4k7, symbol Device:R_Small
- added RN2: 4k7, Resistor_THT:R_Array_SIP9, symbol Device:R_Network08
- added U12: 2716, symbol Custom:2716
- added U2: 74LS138, symbol 74xx:74LS138
- added U6: MC6802, Package_DIP:DIP-40_W15.24mm, symbol CPU_NXP_6800:MC6802
- added Y?: Crystal, symbol Device:Crystal
Connections:
- new net: D?.1 (K), D?.1 (K), LK2.2 (Pin_2)
- new net: C?.1, U6.38 (XTAL), Y?.1
- new net: C?.1, U6.39 (EXTAL), Y?.2
- new net A0: U12.8 (A0), U6.9 (A0)
- new net A1: U12.7 (A1), U6.10 (A1)
- new net A10: U12.19 (A10), U6.19 (A10)
- new net A11: U6.20 (A11)
- new net A12: U6.22 (A12)
- new net A13: U2.1 (A0), U6.23 (A13)
- new net A14: U2.2 (A1), U6.24 (A14)
- new net A15: U2.3 (A2), U6.25 (A15)
- new net A2: U12.6 (A2), U6.11 (A2)
- new net A3: U12.5 (A3), U6.12 (A3)
- new net A4: U12.4 (A4), U6.13 (A4)
- new net A5: U12.3 (A5), U6.14 (A5)
- new net A6: U12.2 (A6), U6.15 (A6)
- new net A7: U12.1 (A7), U6.16 (A7)
- new net A8: U12.23 (A8), U6.17 (A8)
- new net A9: U12.22 (A9), U6.18 (A9)
- new net ACIA_CS: U2.15 (O0)
- new net BA: U6.7 (BA)
- new net CS1: U2.14 (O1)
- new net CS2: U2.13 (O2)
- new net CS3: U2.12 (O3)
- new net CS4: U2.11 (O4)
- new net CS5: U2.10 (O5)
- new net CS6: U2.9 (O6)
- new net CS7: U12.20 (OE), U2.7 (O7)
- new net D0: RN2.2 (R1), U12.9 (D0), U6.33 (D0)
- new net D1: RN2.3 (R2), U12.10 (D1), U6.32 (D1)
- new net D2: RN2.4 (R3), U12.11 (D2), U6.31 (D2)
- new net D3: RN2.5 (R4), U12.13 (D3), U6.30 (D3)
- new net D4: RN2.6 (R5), U12.14 (D4), U6.29 (D4)
- new net D5: D?.2 (A), RN2.7 (R6), U12.15 (D5), U6.28 (D5)
- new net D6: RN2.8 (R7), U12.16 (D6), U6.27 (D6)
- new net D7: D?.2 (A), RN2.9 (R8), U12.17 (D7), U6.26 (D7)
- new net E: U6.37 (E)
- new net GND: C?.2, C?.2, LK2.1 (Pin_1), U12.12 (VEE), U12.18 (CE), U2.4 (E1), U2.5 (E2), U2.8 (GND), U6.1 (VSS), U6.21 (VSS)
- new net MCU1_HLT: R6.2, U6.2 (~{HALT}), U6.3 (MR)
- new net R/~{W}: U6.34 (R/~{W})
- new net VCC: R12.1, R5.1, R6.1, R7.1, RN2.1 (common), U12.21 (VPP), U12.24 (VCC), U2.16 (VCC), U6.35 (VCC_STANDBY), U6.36 (RE), U6.8 (VCC)
- new net VMA: U2.6 (E3), U6.5 (VMA)
- new net ~{IRQ}: R5.2, U6.4 (~{IRQ})
- new net ~{NMI}: R7.2, U6.6 (~{NMI})
- new net ~{RESET}: R12.2, U6.40 (~{RESET})
- no-connect marks 0 -> 6

Commit message: cleanup, fixes, started on power supplies
Parts:
- added C12, C2, C6: .1u, symbol Device:C_Small
- C13, C14: renamed from C?; value C_Small -> 27p
- X1: renamed from Y?; value Crystal -> 4MHz
- gave numbers to parts that had none: 2
- renumbered U12 to IC12, U2 to IC2, U6 to IC6, RN2 to RP2
Connections:
- net GND: now also C12.2, C2.2, C6.2
- net VCC: now also C12.1, C2.1, C6.1
Other:
- moved on the sheet: C13, C14, X1

Commit message: More power supply work
Parts:
- IC2: value 74LS138 -> 74LD138
