File: schematics/secondary_supply.kicad_sch (KiCad schematic)
At the start: 0 parts

Commit message: More power supply work
Changed lines of the file:
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@@
-(kicad_sch (version 20211123) (generator eeschema)
+(kicad_sch (version 20230121) (generator eeschema)
   (paper "A4")
-  (hierarchical_label "MB[1..10]" (shape bidirectional) (at 124.46 99.06 0)
-    (effects (font (size 1.27 1.27)) (justify left))
+  (bus_entry (at 124.46 101.6) (size 2.54 2.54)
+    (stroke (width 0) (type default))
+  )
+  (bus (pts (xy 124.46 99.06) (xy 124.46 101.6))
+    (stroke (width 0) (type default))
+  )
+  (bus (pts (xy 121.92 99.06) (xy 124.46 99.06))
+    (stroke (width 0) (type default))
+  )
+  (bus (pts (xy 124.46 101.6) (xy 124.46 109.22))
+    (stroke (width 0) (type default))
+  )
+  (wire (pts (xy 127 104.14) (xy 129.54 104.14))
+    (stroke (width 0) (type default))
+  )
+  (label "SS3" (at 129.54 104.14 0) (fields_autoplaced)
+    (effects (font (size 1.27 1.27)) (justify left bottom))
+  )
+  (hierarchical_label "SS[1..10]" (shape bidirectional) (at 121.92 99.06 180) (fields_autoplaced)
+    (effects (font (size 1.27 1.27)) (justify right))
   )
 )
